File: aether.kicad_sch (KiCad schematic)
At the start: 64 parts, among them J1 XT30PW-M, J2 USB_C_Receptacle_USB2.0, U1 TPS562201DDCR, U10 SHT45-AD1B-R2, U11 RFM95W-915S2, U12 W25Q128JVSIQ, U2 TPS562201DDCR, U3 DMG3415U-7, U4 USBLC6-2SC6, U5 SAM-M10Q-00B, U6 MS860702BA01-50, U7 DPS310, U8 H3LIS331DL, U9 LSM6DSO32TR

Commit message: Update aether.kicad_sch
Parts:
- added J3: B4B-PH-SM4-TB(LF)(SN), JST_B4B-PH-SM4-TB(LF)(SN), symbol B4B-PH-SM4-TB_LF__SN_:B4B-PH-SM4-TB(LF)(SN)
Connections:
- net FLASH_CLK is gone; now on net DPS310_SCK: U12.6 (CLK)
- net FLASH_SDI is gone; now on net DPS310_SDI/SDA: U12.5 (DI(IO0))
- net FLASH_SDO is gone; now on net DPS310_SDO: U12.2 (DO(IO1))
- net H3LIS331DL_SCK is gone; now on net DPS310_SCK: U8.4 (SCL/SPC)
- net H3LIS331DL_SDI/SDA is gone; now on net DPS310_SDI/SDA: U8.6 (SDA/SDI/SDO)
- net H3LIS331DL_SDO is gone; now on net DPS310_SDO: U8.7 (SDO/SA0)
- net LSM6DSO32TR_SCL is gone; now on net DPS310_SCK: U9.13 (SCL)
- net LSM6DSO32TR_SDA is gone; now on net DPS310_SDI/SDA: U9.14 (SDA)
- net LSM6DSO32TR_SDO is gone; now on net DPS310_SDO: U9.1 (SDO/SA0)
- net MS8607_SCL is gone; now on net GPS_SCL: U6.8 (SCL)
- net MS8607_SDA is gone; now on net GPS_SDA: U6.7 (SDA)
- net SHT45_SCL is gone; now on net GPS_SCL: U10.2 (SCL)
- net SHT45_SDA is gone; now on net GPS_SDA: U10.1 (SDA)
- net 5V: now also J3.1
- net GND: now also J3.2
- new net: J3.SH1 (SHIELD), J3.SH2 (SHIELD)
- new net RFD900_RX: J3.3
- new net RFD900_TX: J3.4
- no-connect marks 3 -> 4
Other:
- note added: "I2C BUS I (MCU)"
- note added: "RFD900 - UART (SCU)"
- note added: "SDI - Serial Data In -> Microcontroller Out Sensor In"
- note added: "SDO - Serial Data Out -> Microcontroller In Sensor Out"
- note added: "SPI BUS I (MCU)"
- note added: "SPI BUS I (SCU)"
- moved on the sheet: D1, J1, R7, R8, U3

Commit message: Update aether.kicad_sch
Parts:
- added U13: STM32F405VGTx, Package_QFP:LQFP-100_14x14mm_P0.5mm, symbol MCU_ST_STM32F4:STM32F405VGTx
- C23: value 100nF -> 10uF
Connections:
- net GND: now also U13.10 (VSS), U13.20 (VSSA), U13.27 (VSS), U13.74 (VSS), U13.99 (VSS)
- new net F405_VDD: U13.100 (VDD), U13.11 (VDD), U13.19 (VDD), U13.28 (VDD), U13.50 (VDD), U13.6 (VBAT), U13.75 (VDD)
- new net F405_VDDA: U13.22 (VDDA)
Other:
- note added: "MCU - STM32 (F405)"
- moved on the sheet: D1, J1, R7, R8, U3

Commit message: Added ESP32 + Modified Symbols
Parts:
- removed J3: B4B-PH-SM4-TB(LF)(SN), JST_B4B-PH-SM4-TB(LF)(SN), symbol B4B-PH-SM4-TB_LF__SN_:B4B-PH-SM4-TB(LF)(SN)
- removed U13: STM32F405VGTx, Package_QFP:LQFP-100_14x14mm_P0.5mm, symbol MCU_ST_STM32F4:STM32F405VGTx
- added C24, C25, C26, C27, C28, C29, C30: 100nF, Capacitor_SMD:C_0201_0603Metric, symbol Device:C
- added IC1: ESP32-S3-MINI-1U-N8, ESP32S3MINI1UN8, symbol ESP32-S3-MINI-1U-N8:ESP32-S3-MINI-1U-N8
- added J3, J6, J7: SM04B-SRSS-TB(LF)(SN), JST_SM04B-SRSS-TB(LF)(SN), symbol SM04B-SRSS-TB_LF__SN_:SM04B-SRSS-TB(LF)(SN)
- added J4: USB_C_Receptacle_USB2.0, symbol Connector:USB_C_Receptacle_USB2.0
- added J5: Micro_SD_Card, symbol Connector:Micro_SD_Card
- added R22, R23: 5.1k, Resistor_SMD:R_0201_0603Metric, symbol Device:R
- added U14: STM32F405VGTx, Package_QFP:LQFP-100_14x14mm_P0.5mm, symbol MCU_ST_STM32F4:STM32F405VGTx
- added U15: USBLC6-2SC6, Package_TO_SOT_SMD:SOT-23-6, symbol Power_Protection:USBLC6-2SC6
Connections:
- net 3.3V: now also C24.1, C25.1, C26.1, C27.1, C28.1, C29.1, C30.1, IC1.3 (3V3), U14.11 (VDD), U14.19 (VDD), U14.28 (VDD), U14.6 (VBAT)
- net 5V: now also J3.1
- net DPS310_SCK: now also U14.30 (PA5), U14.52 (PB13)
- net DPS310_SDI/SDA: now also U14.18 (PC3), U14.32 (PA7), U14.54 (PB15)
- net DPS310_SDO: now also U14.17 (PC2), U14.31 (PA6), U14.53 (PB14)
- net F405_VDDA: now also U14.22 (VDDA)
- net GND: now also C24.2, C25.2, C26.2, C27.2, C28.2, C29.2, C30.2, IC1.1 (GND_1), IC1.2 (GND_2), IC1.42 (GND_3), IC1.43 (GND_4), IC1.46 (GND_5), IC1.47 (GND_6), IC1.48 (GND_7), IC1.49 (GND_8), IC1.50 (GND_9), IC1.51 (GND_10), IC1.52 (GND_11), IC1.53 (GND_12), IC1.54 (GND_13), IC1.55 (GND_14), IC1.56 (GND_15), IC1.57 (GND_16), IC1.58 (GND_17), IC1.59 (GND_18), IC1.60 (GND_19), IC1.61 (GND_20), IC1.62 (GND_21), IC1.63 (GND_22), IC1.64 (GND_23), IC1.65 (GND_24), IC1.66 (GND_25), IC1.67 (GND_26), IC1.68 (GND_27), IC1.69 (GND_28), IC1.70 (GND_29), IC1.71 (GND_30), IC1.72 (GND_31), IC1.73 (GND_32), J3.2, J4.A1 (GND), J4.A12 (GND), J4.B1 (GND), J4.B12 (GND), R22.1, R23.2, U14.10 (VSS), U14.20 (VSSA), U14.27 (VSS), U14.74 (VSS), U14.99 (VSS), U15.2 (GND)
- net GPS_SCL: now also U14.92 (PB6)
- net GPS_SDA: now also U14.93 (PB7)
- net RFD900_RX: now also J3.3
- net RFD900_TX: now also J3.4
- net VBAT: no longer J2.A4 (VBUS), J2.A9 (VBUS), J2.B4 (VBUS), J2.B9 (VBUS)
- net VBUS: now also U15.5 (VBUS)
- net BOARD_D+ renamed STM32_D+
- net BOARD_D- renamed STM32_D-
- net D+ renamed USB1_D+
- net D- renamed USB1_D-
- new net: J3.S1 (SHIELD), J3.S2 (SHIELD)
- new net: J7.S1 (SHIELD), J7.S2 (SHIELD)
- new net: J6.S1 (SHIELD), J6.S2 (SHIELD)
- new net: J4.A4 (VBUS), J4.A9 (VBUS), J4.B4 (VBUS), J4.B9 (VBUS)
- new net: J4.A5 (CC1), R22.2
- new net: J4.B5 (CC2), R23.1
- new net: J2.A4 (VBUS), J2.A9 (VBUS), J2.B4 (VBUS), J2.B9 (VBUS)
- new net ESP-EN: IC1.45 (EN)
- new net ESP-I2C1_SCL: IC1.9 (IO5)
- new net ESP-I2C1_SDA: IC1.8 (IO4)
- new net ESP-I2C2_SCL: IC1.11 (IO7)
- new net ESP-I2C2_SDA: IC1.10 (IO6)
- new net ESP-RX0: IC1.40 (RXD0)
- new net ESP-RX1: IC1.22 (IO18)
- new net ESP-RX2: IC1.20 (IO16)
- new net ESP-SPI1_CS0: IC1.14 (IO10)
- new net ESP-SPI1_MISO: IC1.17 (IO13)
- new net ESP-SPI1_MOSI: IC1.15 (IO11)
- new net ESP-SPI1_SCK: IC1.16 (IO12)
- new net ESP-SPI2_CS0: IC1.29 (IO34)
- new net ESP-SPI2_MISO: IC1.33 (IO37)
- new net ESP-SPI2_MOSI: IC1.31 (IO35)
- new net ESP-SPI2_RFM1: IC1.30 (IO48)
- new net ESP-SPI2_RFM2: IC1.34 (IO38)
- new net ESP-SPI2_SCK: IC1.32 (IO36)
- new net ESP-TX0: IC1.39 (TXD0)
- new net ESP-TX1: IC1.21 (IO17)
- new net ESP-TX2: IC1.19 (IO15)
- new net ESP-USB_D+: IC1.24 (IO20)
- new net ESP-USB_D-: IC1.23 (IO19)
- new net ESP32_D+: U15.4 (I/O2)
- new net ESP32_D-: U15.6 (I/O1)
- new net F405_VDD4: U14.50 (VDD)
- new net F405_VDD5: U14.75 (VDD)
- new net F405_VDD6: U14.100 (VDD)
- new net I2C2_SCL: U14.47 (PB10)
- new net I2C2_SDA: U14.48 (PB11)
- new net I2C3_SCL: U14.66 (PC9)
- new net I2C3_SDA: U14.67 (PA8)
- new net SPI3_MISO: U14.90 (PB4)
- new net SPI3_MOSI: U14.91 (PB5)
- new net SPI3_SCK: U14.89 (PB3)
- new net UART4_RX: U14.24 (PA1)
- new net UART4_TX: U14.23 (PA0)
- new net UART5_RX: U14.83 (PD2)
- new net UART5_TX: U14.80 (PC12)
- new net USB2_D+: J4.A6 (D+), J4.B6 (D+), U15.3 (I/O2)
- new net USB2_D-: J4.A7 (D-), J4.B7 (D-), U15.1 (I/O1)
- no-connect marks 4 -> 7
Other:
- note added: "I2C 1 (STM32)"
- note added: "I2C 2 (ESP32)"
- note added: "I2C 2 (STM32)"
- note added: "I2C 3 (STM32) <-> I2C 1 (ESP32)"
- note added: "MCU - ESP32"
- note added: "Need SD Card"
- note added: "Notes: - Need Pyro Channels, Continuity - Need Voltage Monitoring ADCs - Need Servo Interface - Maybe PWM over I2C - Verify VBUS, VBAT logic - Need Auto Reset/Boot Logic for STM32 and ESP32 on USB"
- note added: "RFD900 - UART (ESP32)"
- note added: "SPI 1 (STM32)"
- note added: "SPI 2 (ESP32)"
- note added: "SPI 2 (STM32)"
- note added: "SPI 3 (STM32) <-> SPI 1 (ESP32)"
- note added: "SPID -> MOSI"
- note added: "SPIQ -> MISO"
- note added: "Strapping Pin"
- note added: "USB-C (ESP32)"
- note added: "USB-C (STM32)"
- note removed: "I2C BUS I (MCU)"
- note removed: "RFD900 - UART (SCU)"
- note removed: "SPI BUS I (MCU)"
- note removed: "SPI BUS I (SCU)"
- note removed: "USB-C (USB 2.0)"
- moved on the sheet: C1, C10, C15, C16, C2, C21, C3, C4, C5, C6, C7, C8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

Commit message: Update aether.kicad_sch
Parts:
- removed C30: 100nF, Capacitor_SMD:C_0201_0603Metric, symbol Device:C
- added C31, C35: 100nF, Capacitor_SMD:C_0201_0603Metric, symbol Device:C
- added C32, C33, C37, C38, C39, C40: 2.2uF, Capacitor_SMD:C_0201_0603Metric, symbol Device:C
- added C34: 1uF, Capacitor_SMD:C_0201_0603Metric, symbol Device:C
- added C36: 10uF, Capacitor_SMD:C_0201_0603Metric, symbol Device:C
- added FB1: 600Ω, symbol Device:FerriteBead
- added J10, J11: SM02B-SRSS-TB(LF)(SN), SM02B-SRSS-TB(LF)(SN), symbol SM02B-SRSS-TB_LF__SN_:SM02B-SRSS-TB(LF)(SN)
- added J8, J9: SM04B-SRSS-TB(LF)(SN), JST_SM04B-SRSS-TB(LF)(SN), symbol SM04B-SRSS-TB_LF__SN_:SM04B-SRSS-TB(LF)(SN)
- added R24, R25, R26, R27, R28, R29, R30: 10k, Resistor_SMD:R_0201_0603Metric, symbol Device:R
- added U13, U17: STM32F405RGTx, Package_QFP:LQFP-64_10x10mm_P0.5mm, symbol MCU_ST_STM32F4:STM32F405RGTx
- added U16: PCA9685BS, Package_DFN_QFN:QFN-28-1EP_6x6mm_P0.65mm_EP4.25x4.25mm, symbol Driver_LED:PCA9685BS
- C29: value 100nF -> 10uF
- R7: value 0.1 -> 0.025
Connections:
- net ESP-RX2 is gone; now on net ESP32-RX2: IC1.20 (IO16)
- net ESP-TX2 is gone; now on net ESP32-TX2: IC1.19 (IO15)
- net F405_VDD4 is gone; now on net 3.3V: U14.50 (VDD)
- net RFM95W_CS is gone; now on net ESP32-SPI1_CS0: R18.2, U11.5 (NSS)
- net RFM95W_SCK is gone; now on net ESP32-SPI1_SCK: U11.4 (SCK)
- net RFM95W_SDI is gone; now on net ESP32-SPI1_MOSI: U11.3 (MOSI)
- net RFM95W_SDO is gone; now on net ESP32-SPI1_MISO: U11.2 (MISO)
- net 3.3V: now also J5.4 (VDD), J6.2, C31.1, C36.1, FB1.2, J8.2, R25.2, R26.2, R27.2, R28.2, R29.2, R30.2, U13.1 (VBAT), U13.19 (VDD), U13.32 (VDD), U13.48 (VDD), U13.64 (VDD), U16.25 (VDD)
- net 5V: now also J7.2, J9.2
- net DPS310_CSB: now also U13.33 (PB12), U17.33 (PB12)
- net DPS310_SCK: now also J5.5 (CLK), U13.34 (PB13), U17.34 (PB13); no longer U12.6 (CLK), U14.30 (PA5), U14.52 (PB13)
- net DPS310_SDI/SDA: now also J5.3 (CMD), U13.11 (PC3), U13.35 (PB14), U17.11 (PC3), U17.35 (PB14); no longer U12.5 (DI(IO0)), U14.18 (PC3), U14.32 (PA7), U14.54 (PB15)
- net DPS310_SDO: now also J5.7 (DAT0), U13.10 (PC2), U13.36 (PB15), U17.10 (PC2), U17.36 (PB15); no longer U12.2 (DO(IO1)), U14.17 (PC2), U14.31 (PA6), U14.53 (PB14)
- net F405_VDDA: now also U14.21 (VREF+), C34.1, C35.1, FB1.1, U13.13 (VDDA)
- net FLASH_CS: now also U13.20 (PA4), U17.20 (PA4)
- net GND: now also J5.6 (VSS), J5.9 (SHIELD), J6.1, J7.1, C31.2, C32.2, C33.2, C34.2, C35.2, C36.2, C37.2, C38.2, C39.2, C40.2, J8.1, J9.1, R24.2, U13.12 (VSSA), U13.18 (VSS), U13.63 (VSS), U16.1 (A3), U16.11 (VSS), U16.2 (A4), U16.21 (A5), U16.22 (EXTCLK), U16.26 (A0), U16.27 (A1), U16.28 (A2), U16.29 (VSS), U17.12 (VSSA), U17.18 (VSS), U17.63 (VSS)
- net GPS_SCL: now also U13.58 (PB6), U17.58 (PB6); no longer U14.92 (PB6)
- net GPS_SDA: now also U13.59 (PB7), U17.59 (PB7); no longer U14.93 (PB7)
- net I2C3_SCL: now also U14.67 (PA8); no longer U14.66 (PC9)
- net I2C3_SDA: now also U14.66 (PC9); no longer U14.67 (PA8)
- net STM32_D+: now also U14.71 (PA12); no longer U4.4 (I/O2)
- net STM32_D-: now also U14.70 (PA11); no longer U4.6 (I/O1)
- net STM32-UART1_RX: now reaches J7.3
- net STM32-UART1_RX: now also U14.69 (PA10), U13.43 (PA10), U17.43 (PA10)
- net STM32-UART1_TX: now reaches J7.4
- net STM32-UART1_TX: now also U14.68 (PA9), U13.42 (PA9), U17.42 (PA9)
- net HSE_IN: now reaches U14.12 (PH0)
- net HSE_OUT: now reaches U14.13 (PH1)
- net NRST: now reaches U14.14 (NRST)
- net ESP32-RX2: now reaches U14.25 (PA2)
- net ESP32-RX2: now also J10.2, U13.16 (PA2), U17.16 (PA2)
- net ESP32-TX2: now reaches U14.26 (PA3)
- net ESP32-TX2: now also J10.1, U13.17 (PA3), U17.17 (PA3)
- net SPI1_CS0: now reaches U14.29 (PA4)
- net at U14.49 (VCAP_1): now also C33.1
- net SPI2_CS0: now reaches U14.51 (PB12)
- net STM32-UART3_TX: now reaches U14.55 (PD8)
- net STM32-UART3_TX: now also U13.51 (PC10), U17.51 (PC10)
- net STM32-UART3_RX: now reaches U14.56 (PD9)
- net STM32-UART3_RX: now also U17.52 (PC11)
- net STM32-UART6_TX: now reaches U14.63 (PC6)
- net STM32-UART6_TX: now also U13.37 (PC6), U17.37 (PC6)
- net STM32-UART6_RX: now reaches U14.64 (PC7)
- net STM32-UART6_RX: now also U13.38 (PC7), U17.38 (PC7)
- net at U14.73 (VCAP_2): now also C32.1
- net BOOT0: now reaches U14.94 (BOOT0)
- net STM32-I2C2_SDA: now reaches J6.3
- net STM32-I2C2_SDA: now also R25.1, U13.30 (PB11), U17.30 (PB11)
- net STM32-I2C2_SCL: now reaches J6.4
- net STM32-I2C2_SCL: now also R26.1, U13.29 (PB10), U17.29 (PB10)
- net SD_CS: now reaches J5.2 (DAT3/CD)
- net ESP-EN: no longer names the net of IC1.45 (EN)
- net ESP-I2C1_SCL renamed ESP32-I2C1_SCL
- net ESP32-I2C1_SCL: now also J8.4, R30.1
- net ESP-I2C1_SDA renamed ESP32-I2C1_SDA
- net ESP32-I2C1_SDA: now also J8.3, R29.1
- net ESP-I2C2_SCL renamed ESP32-I2C2_SCL
- net ESP32-I2C2_SCL: now also R28.1, U13.41 (PA8), U17.41 (PA8)
- net ESP-I2C2_SDA renamed ESP32-I2C2_SDA
- net ESP32-I2C2_SDA: now also R27.1, U13.40 (PC9), U17.40 (PC9)
- net ESP-RX0 renamed ESP32-RX0
- net ESP-RX1 renamed ESP32-RX1
- net ESP32-RX1: now also J9.3
- net ESP-SPI1_CS0 renamed ESP32-SPI1_CS0
- net ESP-SPI1_MISO renamed ESP32-SPI1_MISO
- net ESP-SPI1_MOSI renamed ESP32-SPI1_MOSI
- net ESP-SPI1_SCK renamed ESP32-SPI1_SCK
- net ESP-SPI2_CS0 renamed ESP32-SPI2_CS0
- net ESP32-SPI2_CS0: now also U13.50 (PA15), U17.50 (PA15)
- net ESP-SPI2_MISO renamed ESP32-SPI2_MISO
- net ESP32-SPI2_MISO: now also U13.56 (PB4), U17.56 (PB4)
- net ESP-SPI2_MOSI renamed ESP32-SPI2_MOSI
- net ESP32-SPI2_MOSI: now also U13.57 (PB5), U17.57 (PB5)
- net ESP-SPI2_RFM1: no longer names the net of IC1.30 (IO48)
- net ESP-SPI2_RFM2: no longer names the net of IC1.34 (IO38)
- net ESP-SPI2_SCK renamed ESP32-SPI2_SCK
- net ESP32-SPI2_SCK: now also U13.55 (PB3), U17.55 (PB3)
- net ESP-TX0 renamed ESP32-TX0
- net ESP-TX1 renamed ESP32-TX1
- net ESP32-TX1: now also J9.4
- net ESP-USB_D+ renamed ESP32-USB_D+
- net ESP32-USB_D+: now also J11.2
- net ESP-USB_D- renamed ESP32-USB_D-
- net ESP32-USB_D-: now also J11.1
- net ESP32_D+: no longer names the net of U15.4 (I/O2)
- net ESP32_D-: no longer names the net of U15.6 (I/O1)
- net UART4_RX renamed STM32-UART4_RX
- net STM32-UART4_RX: now also U17.15 (PA1)
- net UART4_TX renamed STM32-UART4_TX
- net STM32-UART4_TX: now also U17.14 (PA0)
- net UART5_RX renamed STM32-UART5_RX
- net STM32-UART5_RX: now also U13.54 (PD2), U17.54 (PD2)
- new net: C37.1, U13.31 (VCAP_1)
- new net: C38.1, U13.47 (VCAP_2)
- new net: J9.S1 (SHIELD), J9.S2 (SHIELD)
- new net: R24.1, U16.20 (~{OE})
- new net: J8.S1 (SHIELD), J8.S2 (SHIELD)
- new net: C40.1, U17.47 (VCAP_2)
- new net: C39.1, U17.31 (VCAP_1)
- new net FLASH_CLK: U12.6 (CLK), U13.21 (PA5), U17.21 (PA5)
- new net FLASH_SDI: U12.5 (DI(IO0)), U13.22 (PA6), U17.22 (PA6)
- new net FLASH_SDO: U12.2 (DO(IO1)), U13.23 (PA7), U17.23 (PA7)
- new net I2C1_SCL: U14.92 (PB6)
- new net I2C1_SDA: U14.93 (PB7)
- new net PCA9685_SCD: U16.24 (SDA)
- new net PCA9685_SCL: U16.23 (SCL)
- new net PWM0: U16.3 (LED0)
- new net PWM1: U16.4 (LED1)
- new net PWM2: U16.5 (LED2)
- new net PWM3: U16.6 (LED3)
- new net PWM4: U16.7 (LED4)
- new net PWM5: U16.8 (LED5)
- new net PWM6: U16.9 (LED6)
- new net PWM7: U16.10 (LED7)
- new net SPI1_MISO: U14.31 (PA6)
- new net SPI1_MOSI: U14.32 (PA7)
- new net SPI1_SCK: U14.30 (PA5)
- new net SPI2_MISO: U14.17 (PC2), U14.53 (PB14)
- new net SPI2_MOSI: U14.18 (PC3), U14.54 (PB15)
- new net SPI2_SCK: U14.52 (PB13)
- new net STM32-BOOT0: U13.7 (NRST), U17.7 (NRST)
- new net STM32-HSE_IN: U13.5 (PH0), U17.5 (PH0)
- new net STM32-HSE_OUT: U13.6 (PH1), U17.6 (PH1)
- new net STM32-NRST: U13.60 (BOOT0), U17.60 (BOOT0)
- new net STM32-UART5_TX: U17.53 (PC12)
- new net STM32_USB_D+: U13.45 (PA12), U17.45 (PA12)
- new net STM32_USB_D-: U13.44 (PA11), U17.44 (PA11)
- no-connect marks 7 -> 21
Other:
- note added: "3.3V Buck Converter"
- note added: "5V Buck Converter"
- note added: "I2C 1 (ESP32)"
- note added: "I2C 3 (STM32) - I2C 2 (ESP32)"
- note added: "MCU - STM32"
- note added: "MCU Decoupling Caps"
- note added: "Need to change I2C address"
- note added: "PCA9685 (I2C)"
- note added: "Power Input"
- note added: "RFD UART 1 (ESP32)"
- note added: "RFD UART 1 (STM32)"
- note added: "SD CARD (SPI)"
- note added: "SPI 1 (ESP32)"
- note added: "SPI 3 (STM32) - SPI 2 (ESP32)"
- note added: "Strapping Pins"
- note added: "UART 3 (STM32) - UART 2 (ESP32)"
- note added: "UART2 (STM32)"
- note added: "USB (ESP32)"
- note added: "VBAT/VBUS Logic"
- note removed: "3.3V Buck Converter - 2A"
- note removed: "5V Buck Converter - 2A"
- note removed: "Decoupling Capacitor"
- note removed: "Decoupling Capacitors"
- note removed: "I2C 2 (ESP32)"
- note removed: "I2C 3 (STM32) <-> I2C 1 (ESP32)"
- note removed: "Need SD Card"
- note removed: "SPI 2 (ESP32)"
- note removed: "SPI 3 (STM32) <-> SPI 1 (ESP32)"
- note removed: "Strapping Pin"
- moved on the sheet: BT1, C1, C11, C12, C13, C14, C15, C16, C17, C18, C19, C2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

Commit message: added hierarchal sheets
Parts:
- removed BT1: Battery_Cell, symbol Device:Battery_Cell
- removed C1, C2, C6, C7: 10uF, Capacitor_SMD:C_0805_2012Metric, symbol Device:C
- removed C10, C4, C5, C9: 22uF, Capacitor_SMD:C_0805_2012Metric, symbol Device:C
- removed C11, C12, C13, C15, C16, C17, C18, C19, C20, C21, C22, C3, C31, C8: 100nF, Capacitor_SMD:C_0201_0603Metric, symbol Device:C
- removed C14: 220nF, Capacitor_SMD:C_0201_0603Metric, symbol Device:C
- removed C23, C29, C36: 10uF, Capacitor_SMD:C_0201_0603Metric, symbol Device:C
- removed D1: B5819W-TP, SOD3716X135N, symbol B5819W-TP:B5819W-TP
- removed D2: 0.5A/40V/420mV, symbol Device:D_Schottky
- removed D3: LED, LED_SMD:LED_0201_0603Metric, symbol Device:LED
- removed IC1: ESP32-S3-MINI-1U-N8, ESP32S3MINI1UN8, symbol ESP32-S3-MINI-1U-N8:ESP32-S3-MINI-1U-N8
- removed J1: XT30PW-M, AMASS_XT30PW-M, symbol XT30PW-M:XT30PW-M
- removed J10, J11: SM02B-SRSS-TB(LF)(SN), SM02B-SRSS-TB(LF)(SN), symbol SM02B-SRSS-TB_LF__SN_:SM02B-SRSS-TB(LF)(SN)
- removed J3, J6, J7, J8, J9: SM04B-SRSS-TB(LF)(SN), JST_SM04B-SRSS-TB(LF)(SN), symbol SM04B-SRSS-TB_LF__SN_:SM04B-SRSS-TB(LF)(SN)
- removed J4: USB_C_Receptacle_USB2.0, symbol Connector:USB_C_Receptacle_USB2.0
- removed J5: Micro_SD_Card, symbol Connector:Micro_SD_Card
- removed L1, L2: 3.9uH, symbol Device:L
- removed R1, R4, R8: 100k, Resistor_SMD:R_0201_0603Metric, symbol Device:R
- removed R11, R12: 470, Resistor_SMD:R_0201_0603Metric, symbol Device:R
- removed R13: 3.3k, Resistor_SMD:R_0201_0603Metric, symbol Device:R
- removed R14: 2.2k, Resistor_SMD:R_0201_0603Metric, symbol Device:R
- removed R15, R16, R17, R18, R19, R20, R21, R24, R25, R26, R27, R28, R29, R3, R30, R6: 10k, Resistor_SMD:R_0201_0603Metric, symbol Device:R
- removed R2: 54.9k, Resistor_SMD:R_0201_0603Metric, symbol Device:R
- removed R22, R23: 5.1k, Resistor_SMD:R_0201_0603Metric, symbol Device:R
- removed R5: 33.2k, Resistor_SMD:R_0201_0603Metric, symbol Device:R
- removed R7: 0.025, symbol Device:R
- removed U1, U2: TPS562201DDCR, SOT95P280X110-6N, symbol TPS562201DDCR:TPS562201DDCR
- removed U10: SHT45-AD1B-R2, SHT4X, symbol SHT45-AD1B-R2:SHT45-AD1B-R2
- removed U11: RFM95W-915S2, XCVR_RFM95W-915S2, symbol RFM95W-915S2:RFM95W-915S2
- removed U12: W25Q128JVSIQ, SOIC127P790X216-8N, symbol W25Q128JVSIQ:W25Q128JVSIQ
- removed U15: USBLC6-2SC6, Package_TO_SOT_SMD:SOT-23-6, symbol Power_Protection:USBLC6-2SC6
- removed U16: PCA9685BS, Package_DFN_QFN:QFN-28-1EP_6x6mm_P0.65mm_EP4.25x4.25mm, symbol Driver_LED:PCA9685BS
- removed U3: DMG3415U-7, SOT95P240X105-3N, symbol DMG3415U-7:DMG3415U-7
- removed U5: SAM-M10Q-00B, XCVR_SAM-M10Q-00B, symbol SAM-M10Q-00B:SAM-M10Q-00B
- removed U6: MS860702BA01-50, TE_MS860702BA01-50, symbol MS860702BA01-50:MS860702BA01-50
- removed U7: DPS310, XDCR_DPS310, symbol DPS310:DPS310
- removed U8: H3LIS331DL, QFN300X300X100-16N, symbol H3LIS331DL:H3LIS331DL
- removed U9: LSM6DSO32TR, LGA-14L_2P5X3X0P83_STM, symbol LSM6DSO32TR:LSM6DSO32TR
- added Q1, Q2, Q3, Q4: NPN, symbol Simulation_SPICE:NPN
- added R33, R35, R37, R39: 330Ω, symbol Device:R
- added R34, R36, R38, R40: 10kΩ, symbol Device:R
- added RN1: 270kΩ, symbol Device:R_Pack04
- added RN2: 47kΩ, symbol Device:R_Pack04
Connections:
- net F405_VDDA: no longer U14.21 (VREF+)
- net GND: now also Q1.3 (E), Q2.3 (E), Q3.3 (E), Q4.3 (E), R34.2, R36.2, R38.2, R40.2, RN2.1 (R1.1), RN2.2 (R2.1), RN2.3 (R3.1), RN2.4 (R4.1)
- net ESP32-I2C2_SCL renamed STM32-I2C3_SCL
- net ESP32-I2C2_SDA renamed STM32-I2C3_SDA
- net ESP32-RX2 renamed STM32-UART2_TX
- net ESP32-SPI2_CS0 renamed STM32-SPI3_CS0
- net ESP32-SPI2_MISO renamed STM32-SPI3_MISO
- net ESP32-SPI2_MOSI renamed STM32-SPI3_MOSI
- net ESP32-SPI2_SCK renamed STM32-SPI3_SCK
- net ESP32-TX2 renamed STM32-UART2_RX
- new net: Q4.2 (B), R39.1, R40.1
- new net: Q1.2 (B), R33.1, R34.1
- new net: Q3.2 (B), R37.1, R38.1
- new net: Q2.2 (B), R35.1, R36.1
- new net F405_VREF+: U14.21 (VREF+)
- new net PYRO-TERM_A: Q1.1 (C), RN1.8 (R1.2)
- new net PYRO-TERM_B: Q2.1 (C), RN1.7 (R2.2)
- new net PYRO-TERM_C: Q3.1 (C), RN1.6 (R3.2)
- new net PYRO-TERM_D: Q4.1 (C), RN1.5 (R4.2)
- new net PYRO_A: R33.2
- new net PYRO_B: R35.2
- new net PYRO_C: R37.2
- new net PYRO_D: R39.2
- new net V-TERM_A: RN1.1 (R1.1), RN2.8 (R1.2)
- new net V-TERM_B: RN1.2 (R2.1), RN2.7 (R2.2)
- new net V-TERM_C: RN1.3 (R3.1), RN2.6 (R3.2)
- new net V-TERM_D: RN1.4 (R4.1), RN2.5 (R4.2)
- no-connect marks 21 -> 3
Other:
- added sheet connectors (connectors.kicad_sch)
- added sheet esp32 (esp32.kicad_sch)
- added sheet power (power.kicad_sch)
- added sheet sensors (sensors.kicad_sch)
- added sheet shared_mcu_buses (shared_mcu_buses.kicad_sch)
- note added: "0x40, 0x76"
- note added: "0x41"
- note added: "0x42"
- note added: "0x44"
- note added: "N-Channel MOSFET 30V, 20 - 30 A 3.3V Gate"
- note added: "Notes: -Add header Pins, antenna pins, verify connectors - Verify VBUS, VBAT logic - Need Auto Reset/Boot Logic for STM32 and ESP32 on USB"
- note added: "Pyro Terminals (STM32)"
- note added: "Pyro Voltage & Cont. (STM32)"
- note removed: "3.3V Buck Converter"
- note removed: "5V Buck Converter"
- note removed: "Battery Initial Charge: 2.8-3.3V Initial Battery Capcity: 1.5 mAh Battery Charge Rate: 0.03mA MAX Voff: 2.0V 120 hours charge time from 2.0-3.1V"
- note removed: "DPS310 (BARO) - SPI"
- note removed: "H3LIS331DL (IMU) - SPI"
- note removed: "I2C 1 (ESP32)"
- note removed: "I2C 2 (STM32)"
- note removed: "I2C 3 (STM32) - I2C 2 (ESP32)"
- note removed: "LSM6DSO32TR (IMU) - SPI"
- note removed: "MCU - ESP32"
- note removed: "MS8607 (PHT) - I2C"
- note removed: "Need to change I2C address"
- note removed: "Notes: - Need Pyro Channels, Continuity - Need Voltage Monitoring ADCs - Need Servo Interface - Maybe PWM over I2C - Verify VBUS, VBAT logic - Need Auto Reset/Boot Logic for STM32 and ESP32 on USB"
- note removed: "Only for SPI Mode"
- note removed: "PCA9685 (I2C)"
- note removed: "Power Input"
- note removed: "RFD UART 1 (ESP32)"
- note removed: "RFD UART 1 (STM32)"
- note removed: "RFD900 - UART (ESP32)"
- note removed: "RFM95HCW (RF) - SPI"
- note removed: "SAM-M10Q (GPS) - I2C"
- note removed: "SD CARD (SPI)"
- note removed: "SHT45 (HT) - I2C"
- note removed: "SPI 3 (STM32) - SPI 2 (ESP32)"
- note removed: "SPI CS Pull Up"
- note removed: "SPID -> MOSI"
- note removed: "SPIQ -> MISO"
- note removed: "Strapping Pins"
- note removed: "UART 3 (STM32) - UART 2 (ESP32)"
- note removed: "UART2 (STM32)"
- note removed: "USB (ESP32)"
- note removed: "USB-C (ESP32)"
- note removed: "VBAT/VBUS Logic"
- note removed: "W25Q128 (FLASH) - SPI (QSPI)"
- moved on the sheet: C24, C25, C26, C27, C28, C34, C35, C37, C38, FB1, J2, R10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

Commit message: Organized Schematics & Fixed Notes
Parts:
- added BZ1: Buzzer, symbol Device:Buzzer
- added C36, C41: C, symbol Device:C
- added C42: 100nF, Capacitor_SMD:C_0201_0603Metric, symbol Device:C
- added D4: LED, symbol Device:LED
- added D5: WS2812B, LED_SMD:LED_WS2812B_PLCC4_5.0x5.0mm_P3.2mm, symbol LED:WS2812B
- added Q5: NPN, symbol Simulation_SPICE:NPN
- added R41, R43, R44: R, symbol Device:R
- added R42: 10kΩ, symbol Device:R
- added SW1: SW_SPDT, symbol Switch:SW_SPDT
- added SW3: SW_Push, symbol Switch:SW_Push
- added Y1: 25MHz, symbol Device:Crystal_GND24
Connections:
- net 3.3V: now also BZ1.1 (-), D5.1 (VDD), SW1.1 (A)
- net GND: now also C36.2, C41.1, C42.2, D4.1 (K), D5.3 (VSS), Q5.3 (E), SW1.3 (C), SW3.1, Y1.2, Y1.4
- net STM32-BOOT0: now also R42.1, R43.2
- net STM32-HSE_IN: now also C41.2, Y1.1
- net STM32-HSE_OUT: now also R41.1
- net STM32-NRST: now also C42.1, SW3.2
- new net: C36.1, R41.2, Y1.3
- new net: R42.2, SW1.2 (B)
- new net: BZ1.2 (+), Q5.1 (C)
- new net: Q5.2 (B), R44.1
- new net: D4.2 (A), R43.1
- new net BUZZ_IN: R44.2
- new net STM32-RGB_IN: D5.4 (DIN)
- no-connect marks 3 -> 4
Other:
- removed sheet shared_mcu_buses
- note added: "BOOT0 Switch"
- note added: "Buzzer"
- note added: "Current Limiting R"
- note added: "Do Math To Find CAP and R Values"
- note added: "EMI Filter"
- note added: "HSE Crystal"
- note added: "Notes: - Add header Pins, antenna pins, verify connectors - Verify VBUS, VBAT logic - Need Auto Reset/Boot Logic for STM32 and ESP32 on USB"
- note added: "RGB Led"
- note added: "Reset Switch"
- note removed: "Notes: -Add header Pins, antenna pins, verify connectors - Verify VBUS, VBAT logic - Need Auto Reset/Boot Logic for STM32 and ESP32 on USB"
- company: (none) -> nyuad.space
- title: (none) -> MCU - STM32 Schematic
- moved on the sheet: C24, C25, C26, C27, C28, C32, C33, C34, C35, C37, C38, C39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
