File: shared_mcu_buses.kicad_sch (KiCad schematic)
At the start: 3 parts

Commit message: Organized Schematics & Fixed Notes
Other:
- company: (none) -> nyuad.space
- title: (none) -> Aether Flight Computer
Changed lines of the file:
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@@
 (kicad_sch (version 20230121) (generator eeschema)
   (paper "A4")
+  (title_block
+    (title "Aether Flight Computer")
+    (company "nyuad.space")
+  )
   (junction (at 124.46 81.28) (diameter 0) (color 0 0 0 0)
   )
