File: aether.kicad_pcb (KiCad board)
At the start: 2 copper layers, 153 parts, among them J1 XT30PW-M, Q1 NPN, Q2 CSD17575Q3, Q3 CSD17575Q3, Q4 CSD17575Q3, Q5 CSD17575Q3, Q6 PNP, SW1 TDD01H0SB1R, SW2 PTS526_SM08_SMTR2_LFS, SW3 TDD01H0SB1R, SW4 PTS526_SM08_SMTR2_LFS, U1 USBLC6-2SC6, U10 TPS562201DDCR, U11 TPS562201DDCR, U12 INA219AxD, U2 USBLC6-2SC6, U3 SAM-M10Q-00B, U4 DPS310, U5 H3LIS331DL, U6 LSM6DSO32TR, U7 PCA9685BS, U8 MS860702BA01-50, U9 SHT45-AD1B-R2

Commit message: updated pcb
Parts:
- added ANT1: 5-1814832-1, 5-1814832-1:TE_5-1814832-1, F.Cu at (120.7, 64.7)
- added BZ1: CSS-0575A-SMT, CSS-0575A-SMT:CUI_CSS-0575A-SMT, F.Cu at (120.0, 74.5)
Connections:
- Q1 pad 1: Net-(BZ1-+) -> Net-(Q1-C)
Changed lines of the file:
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@@
   (net 200 "unconnected-(USB2-SBU2-PadB8)")
   (net 201 "unconnected-(USB2-SHIELD-PadS1)")
+  (net 202 "Net-(Q1-C)")
   (footprint "Resistor_SMD:R_0603_1608Metric" (layer "F.Cu")
     (at 99.43 102.58)
@@
       (net 2 "GND") (pinfunction "GND") (pintype "power_in"))
   )
+  (footprint "5-1814832-1:TE_5-1814832-1" (layer "F.Cu")
+    (at 120.72 64.65)
+    (property "Availability" "In Stock")
+    (property "Check_prices" "https://www.snapeda.com/parts/5-1814832-1/TE+Connectivity+AMP+Connectors/view-part/?ref=eda")
+    (property "Comment" "5-1814832-1")
+    (property "Description" "\nConnector SMA JACK STR 50 OHM PCB | TE Connectivity 5-1814832-1\n")
+    (property "EU_RoHS_Compliance" "Compliant with Exemptions")
+    (property "MANUFACTURER" "TE Connectivity")
+    (property "MF" "TE Connectivity")
+    (property "MP" "5-1814832-1")
+    (property "Number_of_Positions" "1")
+    (property "PARTREV" "B1")
+    (property "Package" "None")
+    (property "Price" "None")
+    (property "Purchase-URL" "https://www.snapeda.com/api/url_track_click_mouser/?unipart_id=38815&manufacturer=TE Connectivity&part_name=5-1814832-1&search_term=5-1814832-1")
+    (property "STANDARD" "Manufacturer recommendations")
+    (property "Sheetfile" "sensors.kicad_sch")
+    (property "Sheetname" "sensors")
+    (property "SnapEDA_Link" "https://www.snapeda.com/parts/5-1814832-1/TE+Connectivity+AMP+Connectors/view-part/?ref=snap")
+    (attr through_hole)
+    (fp_text reference "ANT1" (at -0.375105 -4.536315) (layer "F.SilkS")
+        (effects (font (size 1.000291 1.000291) (thickness 0.15)))
+    )
+    (fp_text value "5-1814832-1" (at 5.54505 4.86946) (layer "F.Fab")
+        (effects (font (size 1.000913 1.000913) (thickness 0.15)))
+    )
+    (fp_line (start -3.2 1.3) (end -3.2 -1.3)
+      (stroke (width 0.127) (type solid)) (layer "F.SilkS"))
+    (fp_line (start -1.3 -3.2) (end 1.3 -3.2)
+      (stroke (width 0.127) (type solid)) (layer "F.SilkS"))
+    (fp_line (start 1.3 3.2) (end -1.3 3.2)
+      (stroke (width 0.127) (type solid)) (layer "F.SilkS"))
+    (fp_line (start 3.2 1.3) (end 3.2 -1.3)
+      (stroke (width 0.127) (type solid)) (layer "F.SilkS"))
+    (fp_line (start -3.9 -3.9) (end 3.9 -3.9)
+      (stroke (width 0.05) (type solid)) (layer "F.CrtYd"))
+    (fp_line (start -3.9 3.9) (end -3.9 -3.9)
+      (stroke (width 0.05) (type solid)) (layer "F.CrtYd"))
+    (fp_line (start 3.9 -3.9) (end 3.9 3.9)
+      (stroke (width 0.05) (type solid)) (layer "F.CrtYd"))
+    (fp_line (start 3.9 3.9) (end -3.9 3.9)
+      (stroke (width 0.05) (type solid)) (layer "F.CrtYd"))
+    (fp_line (start -3.2 -3.2) (end 3.2 -3.2)
+      (stroke (width 0.127) (type solid)) (layer "F.Fab"))
+    (fp_line (start -3.2 3.2) (end -3.2 -3.2)
+      (stroke (width 0.127) (type solid)) (layer "F.Fab"))
+    (fp_line (start 3.2 -3.2) (end 3.2 3.2)
+      (stroke (width 0.127) (type solid)) (layer "F.Fab"))
+    (fp_line (start 3.2 3.2) (end -3.2 3.2)
+      (stroke (width 0.127) (type solid)) (layer "F.Fab"))
+    (pad "1" thru_hole circle (at 0 0) (size 2.25 2.25) (drill 1.5) (layers "*.Cu" "*.Mask")
+      (net 1 "RFM95W_ANT") (pinfunction "1") (pintype "passive") (solder_mask_margin 0.102))
+    (pad "2" thru_hole circle (at -2.54 -2.54) (size 2.4 2.4) (drill 1.6) (layers "*.Cu" "*.Mask")
+      (net 2 "GND") (pinfunction "2") (pintype "passive") (solder_mask_margin 0.102))
+    (pad "3" thru_hole circle (at 2.54 -2.54) (size 2.4 2.4) (drill 1.6) (layers "*.Cu" "*.Mask")
+      (net 2 "GND") (pinfunction "2") (pintype "passive") (solder_mask_margin 0.102))
+    (pad "4" thru_hole circle (at -2.54 2.54) (size 2.4 2.4) (drill 1.6) (layers "*.Cu" "*.Mask")
+      (net 2 "GND") (pinfunction "2") (pintype "passive") (solder_mask_margin 0.102))
+    (pad "5" thru_hole circle (at 2.54 2.54) (size 2.4 2.4) (drill 1.6) (layers "*.Cu" "*.Mask")
+      (net 2 "GND") (pinfunction "2") (pintype "passive") (solder_mask_margin 0.102))
+  )
   (footprint "CSD17575Q3:TRANS_CSD17308Q3" (layer "F.Cu")
     (at 66.425 100.73)
@@
     )
   )
+  (footprint "CSS-0575A-SMT:CUI_CSS-0575A-SMT" (layer "F.Cu")
+    (at 120.02 74.45)
+    (property "AVAILABILITY" "Unavailable")
+    (property "Availability" "In Stock")
+    (property "CUI_purchase_URL" "https://www.cuidevices.com/product/audio/buzzers/audio-transducers/css-0575a-smt-tr?utm_source=snapeda.com&utm_medium=referral&utm_campaign=snapedaBOM")
+    (property "Check_prices" "https://www.snapeda.com/parts/CSS-0575A-SMT-TR/CUI+Devices/view-part/?ref=eda")
+    (property "DESCRIPTION" "5 mm, 3 V, 75 dB, Surface Mount _SMT_, Magnetic Audio Transducer Buzzer")
+    (property "Description" "5 mm, 3 V, 76 dB, Surface Mount (SMT), Magnetic Audio Transducer Buzzer")
+    (property "MF" "CUI Devices")
+    (property "MP" "CSS-0575A-SMT-TR")
+    (property "PACKAGE" "None")
+    (property "PRICE" "None")
+    (property "Package" "CUI Devices")
+    (property "Price" "None")
+    (property "Purchase-URL" "https://www.snapeda.com/api/url_track_click_mouser/?unipart_id=5633932&manufacturer=CUI Devices&part_name=CSS-0575A-SMT-TR&search_term=buzzer 3v")
+    (property "Sheetfile" "aether.kicad_sch")
+    (property "Sheetname" "")
+    (property "SnapEDA_Link" "https://www.snapeda.com/parts/CSS-0575A-SMT-TR/CUI+Devices/view-part/?ref=snap")
+    (attr smd)
+    (fp_text reference "BZ1" (at -0.069245 -4.244235) (layer "F.SilkS")
+        (effects (font (size 1.405047 1.405047) (thickness 0.15)))
+    )
+    (fp_text value "CSS-0575A-SMT" (at 10.46766 3.99956) (layer "F.Fab")
+        (effects (font (size 1.406535 1.406535) (thickness 0.15)))
+    )
+    (fp_text user "NC" (at -4.70699 -1.52659) (layer "F.SilkS")
+        (effects (font (size 0.480818 0.480818) (thickness 0.15)))
+    )
+    (fp_text user "+" (at -4.45705 2.54688) (layer "F.SilkS")
+        (effects (font (size 1.002717 1.002717) (thickness 0.15)))
+    )
+    (fp_text user "-" (at 3.56466 2.29157) (layer "F.SilkS")
+        (effects (font (size 1.002433 1.002433) (thickness 0.15)))
+    )
+    (fp_line (start -2.5 -0.71) (end -2.5 0.71)
+      (stroke (width 0.127) (type solid)) (layer "F.SilkS"))
+    (fp_line (start -0.66 -2.5) (end 1.5 -2.5)
+      (stroke (width 0.127) (type solid)) (layer "F.SilkS"))
+    (fp_line (start 0.66 2.5) (end -0.65 2.5)
+      (stroke (width 0.127) (type solid)) (layer "F.SilkS"))
+    (fp_line (start 1.5 -2.5) (end 2.5 -1.5)
+      (stroke (width 0.127) (type solid)) (layer "F.SilkS"))
+    (fp_line (start 2.5 -1.5) (end 2.5 0.7)
+      (stroke (width 0.127) (type solid)) (layer "F.SilkS"))
+    (fp_line (start -3.2 -2.85) (end 3.2 -2.85)
+      (stroke (width 0.05) (type solid)) (layer "F.CrtYd"))
+    (fp_line (start -3.2 2.85) (end -3.2 -2.85)
+      (stroke (width 0.05) (type solid)) (layer "F.CrtYd"))
+    (fp_line (start 3.2 -2.85) (end 3.2 2.85)
+      (stroke (width 0.05) (type solid)) (layer "F.CrtYd"))
+    (fp_line (start 3.2 2.85) (end -3.2 2.85)
+      (stroke (width 0.05) (type solid)) (layer "F.CrtYd"))
+    (fp_line (start -2.5 -2.5) (end 1.5 -2.5)
+      (stroke (width 0.127) (type solid)) (layer "F.Fab"))
+    (fp_line (start -2.5 2.5) (end -2.5 -2.5)
+      (stroke (width 0.127) (type solid)) (layer "F.Fab"))
+    (fp_line (start 1.5 -2.5) (end 2.5 -1.5)
+      (stroke (width 0.127) (type solid)) (layer "F.Fab"))
+    (fp_line (start 2.5 -1.5) (end 2.5 2.5)
+      (stroke (width 0.127) (type solid)) (layer "F.Fab"))
+    (fp_line (start 2.5 2.5) (end -2.5 2.5)
+      (stroke (width 0.127) (type solid)) (layer "F.Fab"))
+    (pad "1" smd rect (at -1.9 1.75) (size 2.1 1.7) (layers "F.Cu" "F.Paste" "F.Mask")
+      (net 5 "3.3V") (pintype "passive") (solder_mask_margin 0.102))
+    (pad "2" smd rect (at 1.9 1.75) (size 2.1 1.7) (layers "F.Cu" "F.Paste" "F.Mask")
+      (net 202 "Net-(Q1-C)") (pintype "passive") (solder_mask_margin 0.102))
+    (pad "3" smd rect (at -1.9 -1.75) (size 2.1 1.7) (layers "F.Cu" "F.Paste" "F.Mask")
+      (solder_mask_margin 0.102))
+  )
   (footprint "Crystal:Crystal_SMD_Abracon_ABM8G-4Pin_3.2x2.5mm" (layer "F.Cu")
     (at 91.68 106.34)
@@
       (stroke (width 0.1) (type solid)) (layer "F.Fab"))
     (pad "1" smd roundrect (at -0.9375 -0.95) (size 1.475 0.6) (layers "F.Cu" "F.Paste" "F.Mask") (roundrect_rratio 0.25)
-      (net 4 "Net-(BZ1-+)") (pinfunction "C") (pintype "open_collector"))
+      (net 202 "Net-(Q1-C)") (pinfunction "C") (pintype "open_collector"))
     (pad "2" smd roundrect (at -0.9375 0.95) (size 1.475 0.6) (layers "F.Cu" "F.Paste" "F.Mask") (roundrect_rratio 0.25)
       (net 78 "Net-(Q1-B)") (pinfunction "B") (pintype "input"))

Commit message: grouped components
Parts:
- removed the ANT1 at (71.2, 61.0)
- removed the BZ1 at (91.3, 114.1)
- moved FB1 343.4 mm to (364.7, 283.3)
- moved C9 339.4 mm to (368.1, 277.9)
- moved C11 339.4 mm to (370.5, 289.0)
- moved R4 314.1 mm to (346.9, 267.5)
- moved R12 311.9 mm to (373.2, 242.0)
- moved D1 309.4 mm to (335.4, 265.0)
- moved SW2 306.2 mm to (327.0, 283.9)
- moved R40 305.5 mm to (297.4, 241.0)
- moved R5 304.7 mm to (343.7, 258.0)
- moved R39 304.5 mm to (297.4, 237.4)
- moved C12 301.8 mm to (333.0, 279.2)
- moved SW1 296.2 mm to (340.4, 263.2)
- moved R15 291.5 mm to (380.0, 242.5)
- moved R16 291.5 mm to (380.0, 244.5)
- moved R18 291.5 mm to (380.0, 246.5)
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Connections:
- PWM1 pad 01: PWM0 -> PWM7
- PWM1 pad 02: 3.3V -> 5V
- PWM1 pad 04: PWM1 -> PWM6
- PWM1 pad 05: 3.3V -> 5V
- PWM1 pad 07: PWM2 -> PWM5
- PWM1 pad 08: 3.3V -> 5V
- PWM1 pad 10: PWM3 -> PWM4
- PWM1 pad 11: 3.3V -> 5V
- PWM1 pad 13: PWM4 -> PWM3
- PWM1 pad 14: 3.3V -> 5V
- PWM1 pad 16: PWM5 -> PWM2
- PWM1 pad 17: 3.3V -> 5V
- PWM1 pad 19: PWM6 -> PWM1
- PWM1 pad 20: 3.3V -> 5V
- PWM1 pad 22: PWM7 -> PWM0
- PWM1 pad 23: 3.3V -> 5V
- U12 pad 3: GPS_SDA -> INA219_SDA
- U12 pad 4: GPS_SCL -> INA219_SCL
Routing:
- net 3.3V: track 0.00 -> 22.3 mm
- net GND: track 0.00 -> 19.3 mm
- net STM32-HSE_IN: track 0.00 -> 10.1 mm
- net Net-(C10-Pad1): track 0.00 -> 3.91 mm
- net Net-(STM1-PB2): track 0.00 -> 2.24 mm
- net Net-(STM1-VCAP_1): track 0.00 -> 2.13 mm
- net STM32-HSE_OUT: track 0.00 -> 2.06 mm
- net Net-(STM1-VCAP_2): track 0.00 -> 2.05 mm
- net LSM6DSO32TR_CS: track 0.00 -> 1.67 mm
- net DPS310_CSB: track 0.00 -> 1.45 mm
Other:
- copper layers 2 -> 4

Commit message: updated tracks
Parts:
- added REF**: MountingHole_3.2mm_M3_Pad_Via, MountingHole:MountingHole_3.2mm_M3_Pad_Via, F.Cu at (197.3, 131.2)
- added REF**: MountingHole_3.2mm_M3_Pad_Via, MountingHole:MountingHole_3.2mm_M3_Pad_Via, F.Cu at (105.9, 79.8)
- added REF**: MountingHole_3.2mm_M3_Pad_Via, MountingHole:MountingHole_3.2mm_M3_Pad_Via, F.Cu at (197.3, 79.9)
- added REF**: MountingHole_3.2mm_M3_Pad_Via, MountingHole:MountingHole_3.2mm_M3_Pad_Via, F.Cu at (106.1, 131.2)
- R22, R26, R28, R34: footprint Resistor_SMD:R_0603_1608Metric -> Resistor_SMD:R_0402_1005Metric
- moved ANT1 221.5 mm to (115.0, 130.8)
- moved C1 209.4 mm to (154.9, 115.2)
- moved R1 209.4 mm to (152.9, 115.1)
- moved C10 209.4 mm to (140.1, 107.9)
- moved C2 209.4 mm to (143.9, 102.9)
- moved C3 209.4 mm to (160.4, 103.4)
- moved C4 209.4 mm to (148.9, 113.9)
- moved C5 209.4 mm to (157.4, 114.9)
- moved C6 209.4 mm to (148.9, 114.9)
- moved C7 209.4 mm to (156.4, 114.9)
- moved C8 209.4 mm to (140.1, 101.9)
- moved HSE1 209.4 mm to (140.1, 104.9)
- moved R3 209.4 mm to (143.6, 105.9)
- moved STM1 209.4 mm to (151.9, 106.7)
- moved RFM2 209.0 mm to (121.9, 132.0), turned to 90 degrees
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Connections:
- RFM1 pad 7: RFM95W_DI4 -> RFM95W_DI5
- RFM2 pad 5: RFM95W_DI4 -> RFM95W_DI5
- U12 pad 3: INA219_SDA -> GPS_SDA
- U12 pad 4: INA219_SCL -> GPS_SCL
Routing:
- net GND: track 19.3 -> 34.2 mm
- net 3.3V: track 22.3 -> 34.5 mm
- net PWM0: track 0.00 -> 9.86 mm
- net PWM7: track 0.00 -> 8.86 mm
- net Net-(USB1-CC1): track 0.00 -> 8.09 mm
- net PWM1: track 0.00 -> 8.03 mm
- net Net-(USB2-CC1): track 0.00 -> 7.85 mm
- net Net-(USB1-CC2): track 0.00 -> 7.57 mm
- net Net-(USB2-CC2): track 0.00 -> 7.50 mm
- net PWM6: track 0.00 -> 6.88 mm
- net GPS_VBCKP: track 0.00 -> 6.43 mm
- net PWM2: track 0.00 -> 6.18 mm
- net USB1_D-: track 0.00 -> 5.30 mm
- net USB2_D-: track 0.00 -> 5.24 mm
- net PWM5: track 0.00 -> 4.95 mm
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Other:
- board outline added: 100.1 x 60.2 mm

Commit message: started routing
Parts:
- C16, C17, C18, C19, C20, C24, C25, C30, C31, R22, R26, R29, R30, R31, R32, R33, U4, U5, U7, U8, U9, W25Q1: moved to B.Cu
- R48, R49: footprint Resistor_SMD:R_0603_1608Metric -> Resistor_SMD:R_0402_1005Metric
- moved C11 293.8 mm to (138.8, 108.4), turned to 180 degrees
- moved FB1 285.1 mm to (138.8, 109.5), turned to 180 degrees
- moved C9 284.9 mm to (137.3, 110.8), turned to 180 degrees
- moved R15 259.8 mm to (157.1, 109.1), turned to -90 degrees
- moved R16 259.5 mm to (158.6, 109.1), turned to -90 degrees
- moved R19 249.0 mm to (167.3, 119.0)
- moved R18 248.6 mm to (167.3, 117.8)
- moved R25 246.9 mm to (193.6, 51.7)
- moved D3 246.9 mm to (193.5, 55.2)
- moved BT1 246.2 mm to (171.7, 89.0)
- moved C23 246.2 mm to (175.7, 87.2)
- moved D4 246.2 mm to (173.9, 80.5)
- moved R27 246.2 mm to (173.9, 84.0)
- moved C21 246.2 mm to (187.4, 78.0)
- moved C22 246.2 mm to (175.7, 84.0)
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Connections:
- PWM1 pad 01: PWM7 -> PWM0
- PWM1 pad 04: PWM6 -> PWM1
- PWM1 pad 07: PWM5 -> PWM2
- PWM1 pad 10: PWM4 -> PWM3
- PWM1 pad 13: PWM3 -> PWM4
- PWM1 pad 16: PWM2 -> PWM5
- PWM1 pad 19: PWM1 -> PWM6
- PWM1 pad 22: PWM0 -> PWM7
- RFM2 pad 1: RFM95W_DI1 -> RFM95W_DI5
- RFM2 pad 2: RFM95W_DI2 -> RFM95W_DI4
- RFM2 pad 4: RFM95W_DI4 -> RFM95W_DI2
- RFM2 pad 5: RFM95W_DI5 -> RFM95W_DI1
Routing:
- net STM32-I2C2_SDA: track 0.00 -> 58.7 mm, vias 0 -> 2
- net STM32-I2C2_SCL: track 0.00 -> 58.4 mm, vias 0 -> 2
- net ESP32-SPI1_CS0: track 0.00 -> 56.7 mm
- net ESP32-SPI1_SCK: track 0.00 -> 55.0 mm, vias 0 -> 2
- net ESP32-SPI1_MISO: track 0.00 -> 54.0 mm, vias 0 -> 2
- net ESP32-SPI1_MOSI: track 0.00 -> 52.0 mm, vias 0 -> 2
- net STM32-UART2_RX: track 0.00 -> 51.3 mm, vias 0 -> 2
- net STM32-UART2_TX: track 0.00 -> 45.6 mm, vias 0 -> 2
- net STM32_USB_D-: track 0.00 -> 26.5 mm, vias 0 -> 2
- net STM32-NRST: track 0.00 -> 26.5 mm, vias 0 -> 2
- net STM32_USB_D+: track 0.00 -> 25.6 mm, vias 0 -> 2
- net STM32-SWCLK: track 0.00 -> 20.8 mm, vias 0 -> 2
- net STM32-SWDIO: track 0.00 -> 19.0 mm
- net ESP32-USB_D-: track 0.00 -> 16.8 mm
- net ESP32-USB_D+: track 0.00 -> 15.5 mm
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
Commit message: more routing
Parts:
- moved R12 233.0 mm to (175.3, 118.8), turned to 90 degrees
- moved R36 6.32 mm to (150.0, 61.6)
- moved R35 6.32 mm to (150.0, 59.1)
- moved R15 4.08 mm to (161.2, 109.2), turned to 90 degrees
- moved R16 3.20 mm to (161.2, 111.1)
- moved C29 1.61 mm to (184.0, 119.3), turned to 180 degrees
- moved Q6 0.25 mm to (127.5, 92.7)
- moved R19 0.15 mm to (167.3, 118.8)
- moved C3 0.10 mm to (156.6, 103.5)
Routing:
- net STM32-NRST: track 26.5 -> 113.6 mm, vias 2 -> 3
- net ESP32-I2C1_SCL: track 0.00 -> 86.8 mm
- net ESP32-I2C1_SDA: track 0.00 -> 84.3 mm
- net ESP32-RX1: track 0.00 -> 77.4 mm, vias 0 -> 2
- net ESP32-TX1: track 0.00 -> 77.1 mm, vias 0 -> 2
- net ESP32-GPIO0: track 0.00 -> 72.2 mm
- net STM32-UART1_RX: track 0.00 -> 69.0 mm, vias 0 -> 2
- net STM32-UART1_TX: track 0.00 -> 66.2 mm, vias 0 -> 2
- net ESP32-SPI2_CS0: track 0.00 -> 39.6 mm, vias 0 -> 2
- net ESP32-EN: track 6.00 -> 38.9 mm
- net STM32-UART3_TX: track 0.00 -> 25.8 mm, vias 0 -> 2
- net STM32-UART3_RX: track 0.00 -> 25.3 mm, vias 0 -> 2
- net ESP32-I2C2_SCL: track 0.00 -> 14.1 mm, vias 0 -> 2
- net ESP32-I2C2_SDA: track 0.00 -> 12.7 mm
- net ESP32-RX2: track 0.00 -> 4.40 mm
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
Commit message: more routing
Parts:
- added J2: Screw_Terminal_01x04, TerminalBlock_TE-Connectivity:TerminalBlock_TE_282834-4_1x04_P2.54mm_Horizontal, F.Cu at (158.5, 77.7)
- added RFM3: Conn_01x05_Pin, Connector_PinHeader_1.27mm:PinHeader_1x05_P1.27mm_Vertical, F.Cu at (187.1, 77.0)
- C14, C26, C27, Q2, Q3, Q4, Q5, R10, R11, R23, R24, R28, R37, R38, R8, R9, RN1, RN2, RN3, U6: moved to B.Cu
- U7: value PCA9685BS -> PCA9685PW; footprint Package_DFN_QFN:QFN-28-1EP_6x6mm_P0.65mm_EP4.25x4.25mm -> Package_SO:TSSOP-28_4.4x9.7mm_P0.65mm
- moved C30 280.7 mm to (238.2, 114.3)
- moved U8 280.7 mm to (235.3, 115.6)
- moved C31 263.5 mm to (254.8, 114.6), turned to 0 degrees
- moved U9 263.2 mm to (254.8, 116.5), turned to 90 degrees
- moved BZ1 262.5 mm to (157.4, 86.4)
- moved R2 257.9 mm to (147.8, 94.9), turned to 180 degrees
- moved Q1 257.5 mm to (152.1, 95.5)
- moved R11 250.6 mm to (168.0, 87.0)
- moved C12 249.3 mm to (142.7, 118.2)
- moved R10 246.0 mm to (164.1, 87.0)
- moved Q5 243.1 mm to (168.1, 83.9), turned to 90 degrees
- moved R9 241.5 mm to (160.2, 87.0)
- moved Q4 237.6 mm to (164.2, 83.9), turned to 90 degrees
- moved RN1 237.0 mm to (153.1, 88.2), turned to 180 degrees
- moved R8 237.0 mm to (156.3, 87.0)
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Connections:
- ESP1 pad 18: unconnected-(ESP1-IO14-Pad18) -> RFM95W_DI0
- Q2 pad 5-8: (no net) -> PYRO-TERM_A
- RN1 pad 1: Net-(Q5-G) -> Net-(Q2-G)
- RN1 pad 2: Net-(Q4-G) -> Net-(Q3-G)
- RN1 pad 3: Net-(Q3-G) -> Net-(Q4-G)
- RN1 pad 4: Net-(Q2-G) -> Net-(Q5-G)
- RN2 pad 5: V-TERM_D -> V-TERM_A
- RN2 pad 6: V-TERM_C -> V-TERM_B
- RN2 pad 7: V-TERM_B -> V-TERM_C
- RN2 pad 8: V-TERM_A -> V-TERM_D
- RN3 pad 1: V-TERM_A -> V-TERM_D
- RN3 pad 2: V-TERM_B -> V-TERM_C
- RN3 pad 3: V-TERM_C -> V-TERM_B
- RN3 pad 4: V-TERM_D -> V-TERM_A
- RN3 pad 5: PYRO-TERM_D -> PYRO-TERM_A
- RN3 pad 6: PYRO-TERM_C -> PYRO-TERM_B
- RN3 pad 7: PYRO-TERM_B -> PYRO-TERM_C
- RN3 pad 8: PYRO-TERM_A -> PYRO-TERM_D
- U7 pad 1: GND -> Net-(U7-A0)
- U7 pad 10: PWM7 -> PWM4
- U7 pad 11: GND -> PWM5
- U7 pad 12: unconnected-(U7-LED10-Pad14) -> PWM6
- U7 pad 13: unconnected-(U7-LED10-Pad14) -> PWM7
- U7 pad 14: unconnected-(U7-LED10-Pad14) -> GND
- U7 pad 15: unconnected-(U7-LED10-Pad14) -> unconnected-(U7-LED10-Pad17)
- U7 pad 16: unconnected-(U7-LED10-Pad14) -> unconnected-(U7-LED10-Pad17)
- U7 pad 17: unconnected-(U7-LED10-Pad14) -> unconnected-(U7-LED10-Pad17)
- U7 pad 18: unconnected-(U7-LED10-Pad14) -> unconnected-(U7-LED10-Pad17)
- U7 pad 19: unconnected-(U7-LED10-Pad14) -> unconnected-(U7-LED10-Pad17)
- U7 pad 20: Net-(U7-~{OE}) -> unconnected-(U7-LED10-Pad17)
- U7 pad 21: GND -> unconnected-(U7-LED10-Pad17)
- U7 pad 22: GND -> unconnected-(U7-LED10-Pad17)
- U7 pad 23: GPS_SCL -> Net-(U7-~{OE})
- U7 pad 24: PCA9685_SCD -> GND
- U7 pad 25: 3.3V -> GND
- U7 pad 26: Net-(U7-A0) -> GPS_SCL
- U7 pad 27: GND -> GPS_SDA
- U7 pad 28: GND -> 3.3V
- U7 pad 3: PWM0 -> GND
- U7 pad 4: PWM1 -> GND
- U7 pad 5: PWM2 -> GND
- U7 pad 6: PWM3 -> PWM0
- U7 pad 7: PWM4 -> PWM1
- U7 pad 8: PWM5 -> PWM2
- U7 pad 9: PWM6 -> PWM3
Routing:
- net 5V: track 6.06 -> 178.6 mm
- net GPS_SDA: track 0.00 -> 94.6 mm, vias 0 -> 2
- net GPS_SCL: track 0.00 -> 90.7 mm, vias 0 -> 3
- net STM32-BOOT0: track 0.00 -> 64.5 mm, vias 0 -> 3
- net RFM95W_DI0: track 0.00 -> 47.5 mm
- net Net-(SW1-C): track 0.00 -> 22.3 mm
- net ESP32-EN: track 38.9 -> 59.4 mm, vias 0 -> 2
- net GPS_SAFE: track 0.00 -> 17.7 mm, vias 0 -> 1
- net Net-(Q5-G): track 0.00 -> 15.9 mm
- net Net-(Q4-G): track 0.00 -> 11.6 mm
- net PULSE: track 0.04 -> 11.5 mm
- net PYRO-TERM_D: track 0.00 -> 11.3 mm, vias 0 -> 1
- net PYRO-TERM_A: track 0.00 -> 11.3 mm, vias 0 -> 1
- net PYRO-TERM_B: track 0.00 -> 10.8 mm, vias 0 -> 1
- net PYRO-TERM_C: track 0.00 -> 10.8 mm, vias 0 -> 1
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Other:
- board size 100.1 x 60.2 mm -> 200.2 x 60.4 mm

Commit message: more routing
Parts:
- moved C31 99.5 mm to (156.6, 98.9)
- moved U9 99.5 mm to (156.6, 100.7)
- moved R30 99.2 mm to (120.0, 109.7)
- moved R29 99.2 mm to (122.6, 109.7)
- moved C24 99.2 mm to (119.9, 123.0)
- moved R33 99.2 mm to (121.5, 123.0)
- moved W25Q1 99.2 mm to (122.0, 116.4)
- moved C26 80.9 mm to (159.3, 117.6)
- moved C27 80.9 mm to (159.3, 115.9)
- moved R28 80.9 mm to (156.0, 118.9)
- moved U6 80.9 mm to (156.6, 116.4)
- moved R4 74.2 mm to (149.2, 126.2), turned to -90 degrees
- moved D1 70.0 mm to (151.2, 126.2), turned to 90 degrees
- moved C30 69.2 mm to (171.0, 98.0), turned to 0 degrees
- moved U8 65.3 mm to (171.7, 100.7), turned to -90 degrees
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Connections:
- Q2 pad 5-8: PYRO-TERM_A -> (no net)
- USB1 pad A4: Net-(USB1-VBUS-PadA4) -> VBUS
- USB1 pad A9: Net-(USB1-VBUS-PadA4) -> VBUS
- USB1 pad B4: Net-(USB1-VBUS-PadA4) -> VBUS
- USB1 pad B9: Net-(USB1-VBUS-PadA4) -> VBUS
- USB2 pad A4: Net-(USB2-VBUS-PadA4) -> VBUS
- USB2 pad A9: Net-(USB2-VBUS-PadA4) -> VBUS
- USB2 pad B4: Net-(USB2-VBUS-PadA4) -> VBUS
- USB2 pad B9: Net-(USB2-VBUS-PadA4) -> VBUS
Routing:
- net DPS310_SDI/SDA: track 0.00 -> 54.3 mm, vias 0 -> 2
- net DPS310_SCK: track 0.00 -> 51.9 mm, vias 0 -> 2
- net DPS310_SDO: track 0.00 -> 51.7 mm, vias 0 -> 2
- net SD_CS: track 0.00 -> 48.0 mm, vias 0 -> 2
- net VBUS: track 0.00 -> 43.6 mm, vias 0 -> 4
- net FLASH_CS: track 0.00 -> 37.2 mm, vias 0 -> 2
- net FLASH_SDO: track 0.00 -> 33.9 mm, vias 0 -> 2
- net FLASH_CLK: track 0.00 -> 32.7 mm, vias 0 -> 2
- net FLASH_SDI: track 0.00 -> 32.0 mm, vias 0 -> 2
- net LSM6DSO32TR_CS: track 2.22 -> 17.8 mm, vias 0 -> 1
- net ESP32-GPIO0: track 71.0 -> 84.0 mm
- net GPS_SCL: track 90.7 -> 102.2 mm, vias 3 -> 7
- net GPS_SDA: track 94.6 -> 103.0 mm
- net GND: track 44.2 -> 51.6 mm
- net Net-(U10-VFB): track 1.47 -> 7.93 mm, vias 0 -> 2
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Other:
- board size 200.2 x 60.4 mm -> 100.1 x 60.2 mm
