File: power.kicad_sch (KiCad schematic)
At the start: 33 parts, among them Q6 PNP

Commit message: significant amount of routing done
Parts:
- R51, R52: footprint Resistor_SMD:R_0603_1608Metric -> Resistor_SMD:R_0402_1005Metric
Changed lines of the file:
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@@
       (effects (font (size 1.27 1.27)) (justify left))
     )
-    (property "Footprint" "Resistor_SMD:R_0603_1608Metric" (at 266.192 68.58 90)
+    (property "Footprint" "Resistor_SMD:R_0402_1005Metric" (at 266.192 68.58 90)
       (effects (font (size 1.27 1.27)) hide)
     )
@@
       (effects (font (size 1.27 1.27)) (justify left))
     )
-    (property "Footprint" "Resistor_SMD:R_0603_1608Metric" (at 243.332 68.58 90)
-      (effects (font (size 1.27 1.27)) hide)
-    )
+    (property "Footprint" "Resistor_SMD:R_0402_1005Metric" (at 243.332 68.58 90)
+      (effects (font (size 1.27 1.27)) hide)
+    )

Commit message: added power planes
Parts:
- R51, R52: footprint Resistor_SMD:R_0402_1005Metric -> Resistor_SMD:R_0603_1608Metric
Changed lines of the file:
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@@
       (effects (font (size 1.27 1.27)) (justify left))
     )
-    (property "Footprint" "Resistor_SMD:R_0402_1005Metric" (at 266.192 68.58 90)
+    (property "Footprint" "Resistor_SMD:R_0603_1608Metric" (at 266.192 68.58 90)
       (effects (font (size 1.27 1.27)) hide)
     )
@@
       (effects (font (size 1.27 1.27)) (justify left))
     )
-    (property "Footprint" "Resistor_SMD:R_0402_1005Metric" (at 243.332 68.58 90)
-      (effects (font (size 1.27 1.27)) hide)
-    )
+    (property "Footprint" "Resistor_SMD:R_0603_1608Metric" (at 243.332 68.58 90)
+      (effects (font (size 1.27 1.27)) hide)
+    )
