File: hardware/sensors-2.kicad_sch (KiCad schematic)
At the start: 13 parts, among them U13 BNO086, Y1 32.768kHz

Commit message: rev2 component placement
Parts:
- C43, C46, C47: footprint (none) -> Capacitor_SMD:C_0402_1005Metric
- C44, C45: footprint (none) -> Capacitor_SMD:C_0603_1608Metric
- R56, R57, R58, R59, R60, R61: footprint (none) -> Resistor_SMD:R_0402_1005Metric
- U13: footprint (none) -> Package_LGA:LGA-28_5.2x3.8mm_P0.5mm
- Y1: footprint (none) -> Crystal:Crystal_SMD_3215-2Pin_3.2x1.5mm
